File: PCB/SpringReverbBack.brd (EAGLE design)
At the start: 95 x 28 mm, 43 parts, among them IC4_DRV_RCVR TL072

Commit message: Updated to Eagle 7.2
Parts:
- renumbered TO:INPUT to TO_INPUT, TO:OUTPUT to TO_OUTPUT
Changed lines of the file:
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@@
 <?xml version="1.0" encoding="utf-8"?>
 <!DOCTYPE eagle SYSTEM "eagle.dtd">
-<eagle version="6.4">
+<eagle version="7.2.0">
 <drawing>
 <settings>
@@
 <pass name="Default">
 <param name="RoutingGrid" value="25mil"/>
+<param name="AutoGrid" value="1"/>
+<param name="Efforts" value="0"/>
+<param name="TopRouterVariant" value="1"/>
 <param name="tpViaShape" value="round"/>
 <param name="PrefDir.1" value="-"/>
@@
 <attribute name="VALUE" x="36.59340625" y="24.3181" size="0.8128" layer="27" rot="R90"/>
 </element>
-<element name="TO:INPUT" library="con-lumberg" package="BTOR1" value="TO_TANK" x="12.7" y="21.59" smashed="yes" rot="MR315">
+<element name="TO_INPUT" library="con-lumberg" package="BTOR1" value="TO_TANK" x="12.7" y="21.59" smashed="yes" rot="MR315">
 <attribute name="OC_NEWARK" value="96K7172" x="5.5158" y="1.833434375" size="1.778" layer="28" rot="MR315" display="off"/>
 <attribute name="MPN" value="BTOR 1" x="5.5158" y="1.833434375" size="1.778" layer="28" rot="MR315" display="off"/>
@@
 <element name="R3" library="TomW" package="0207/10" value="2.2k" x="24.13" y="20.32"/>
 <element name="C3" library="TomW" package="C050-024X044" value="10n" x="21.59" y="22.86" rot="R180"/>
-<element name="TO:OUTPUT" library="con-lumberg" package="BTOR1" value="FROM_TANK" x="12.7" y="6.35" smashed="yes" rot="MR45">
+<element name="TO_OUTPUT" library="con-lumberg" package="BTOR1" value="FROM_TANK" x="12.7" y="6.35" smashed="yes" rot="MR45">
 <attribute name="OC_NEWARK" value="96K7172" x="12.7" y="6.35" size="1.778" layer="28" rot="MR45" display="off"/>
 <attribute name="MPN" value="BTOR 1" x="12.7" y="6.35" size="1.778" layer="28" rot="MR45" display="off"/>
@@
 <signals>
 <signal name="N$4">
-<contactref element="TO:INPUT" pad="S"/>
+<contactref element="TO_INPUT" pad="S"/>
 <contactref element="C3" pad="2"/>
 <contactref element="IC4_DRV_RCVR" pad="1"/>
@@
 </signal>
 <signal name="N$7">
-<contactref element="TO:OUTPUT" pad="T"/>
+<contactref element="TO_OUTPUT" pad="T"/>
 <contactref element="IC4_DRV_RCVR" pad="5"/>
 <contactref element="R5" pad="2"/>
@@
 </signal>
 <signal name="N$5">
-<contactref element="TO:INPUT" pad="T"/>
+<contactref element="TO_INPUT" pad="T"/>
 <contactref element="C2" pad="1"/>
 <contactref element="R3" pad="1"/>
@@
 <contactref element="R5" pad="1"/>
 <contactref element="R4" pad="2"/>
-<contactref element="TO:OUTPUT" pad="S"/>
+<contactref element="TO_OUTPUT" pad="S"/>
 <contactref element="D3" pad="C"/>
 <contactref element="D4" pad="A"/>
